File: hardware/espac.kicad_pcb (KiCad board)
At the start: 2 copper layers, 90 x 90 mm, 43 parts, among them J1 USB_C_Receptacle_USB2.0_14P, J2 A3144, J3 A3144, J4 Conn_01x07, J5 Conn_01x10, J6 Conn_01x10, J7 Conn_01x02, Q1 TEMT6000, SW1 RESET, SW2 BOOT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

Commit message: pcb changes
Parts:
- removed J6: Conn_01x10, Connector_PinSocket_2.54mm:PinSocket_1x10_P2.54mm_Vertical
- added C13: 100nF, Capacitor_SMD:C_0805_2012Metric_Pad1.18x1.45mm_HandSolder, F.Cu at (235.0, 86.7)
- added C14: 100nF, Capacitor_SMD:C_0805_2012Metric_Pad1.18x1.45mm_HandSolder, F.Cu at (224.2, 89.6)
- added C15: 100nF, Capacitor_SMD:C_0805_2012Metric_Pad1.18x1.45mm_HandSolder, F.Cu at (216.3, 97.5)
- added C16: 100nF, Capacitor_SMD:C_0805_2012Metric_Pad1.18x1.45mm_HandSolder, F.Cu at (213.4, 108.2)
- added C17: 100nF, Capacitor_SMD:C_0805_2012Metric_Pad1.18x1.45mm_HandSolder, F.Cu at (216.3, 119.0)
- added C18: 100nF, Capacitor_SMD:C_0805_2012Metric_Pad1.18x1.45mm_HandSolder, F.Cu at (224.2, 126.9)
- added D10: SK6812SIDE-A, sk6812:SK6812-SIDE-A, F.Cu at (217.6, 100.3)
- added D11: SK6812SIDE-A, sk6812:SK6812-SIDE-A, F.Cu at (216.0, 110.1)
- added D12: SK6812SIDE-A, sk6812:SK6812-SIDE-A, F.Cu at (219.4, 119.3)
- added D13: SK6812SIDE-A, sk6812:SK6812-SIDE-A, F.Cu at (227.0, 125.6)
- added D8: SK6812SIDE-A, sk6812:SK6812-SIDE-A, F.Cu at (233.1, 89.3)
- added D9: SK6812SIDE-A, sk6812:SK6812-SIDE-A, F.Cu at (223.9, 92.7)
- moved D5 104.1 mm to (253.9, 106.4), turned to -90 degrees
- moved D4 103.2 mm to (252.3, 116.2), turned to -120 degrees
- moved D6 102.0 mm to (250.5, 97.2), turned to -60 degrees
- moved D3 99.5 mm to (246.0, 123.8), turned to -150 degrees
- moved D7 97.4 mm to (242.9, 90.9), turned to -30 degrees
- moved C10 96.7 mm to (256.5, 108.2), turned to -90 degrees
- moved C9 95.6 mm to (253.6, 119.0), turned to -120 degrees
- moved C11 93.9 mm to (253.6, 97.5), turned to -60 degrees
- moved D2 93.4 mm to (236.8, 127.2)
- moved C8 92.4 mm to (245.7, 126.9), turned to -150 degrees
- moved C12 87.8 mm to (245.7, 89.6), turned to -30 degrees
- moved C7 83.4 mm to (235.0, 129.8), turned to 180 degrees
- moved R7 37.6 mm to (157.7, 110.5), turned to -90 degrees
- moved R6 36.8 mm to (157.7, 101.6), turned to -90 degrees
- moved J3 30.6 mm to (152.7, 110.5), turned to -90 degrees
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Connections:
- D7 pad 3: unconnected-(D7-DOUT-Pad3) -> Net-(D7-DOUT)
- J5 pad 1: /GPIO_1 -> /GPIO_TX
- J5 pad 2: /GPIO_8 -> /GPIO_RX
- U1 pad 10: /GPIO_17 -> unconnected-(U1-IO17-Pad10)
- U1 pad 15: /GPIO_3 -> unconnected-(U1-IO3-Pad15)
- U1 pad 16: /GPIO_46 -> unconnected-(U1-IO46-Pad16)
- U1 pad 23: /GPIO_21 -> unconnected-(U1-IO21-Pad23)
- U1 pad 26: /GPIO_45 -> unconnected-(U1-IO45-Pad26)
- U1 pad 31: /GPIO_38 -> unconnected-(U1-IO38-Pad31)
- U1 pad 32: /GPIO_39 -> unconnected-(U1-IO39-Pad32)
- U1 pad 33: /GPIO_40 -> unconnected-(U1-IO40-Pad33)
- U1 pad 34: /GPIO_41 -> unconnected-(U1-IO41-Pad34)
- U1 pad 35: /GPIO_42 -> unconnected-(U1-IO42-Pad35)
- U1 pad 39: /GPIO_1 -> unconnected-(U1-IO1-Pad39)
Routing:
- net +3.3V: track 115.1 -> 312.7 mm, vias 2 -> 6
- net /GPIO_21: track 147.9 -> 0.00 mm, vias 8 -> 0
- net /GPIO_42: track 128.9 -> 0.00 mm, vias 4 -> 0
- net /GPIO_1: track 126.2 -> 0.00 mm, vias 4 -> 0
- net /GPIO_38: track 123.6 -> 0.00 mm, vias 4 -> 0
- net /GPIO_40: track 123.1 -> 0.00 mm, vias 4 -> 0
- net /GPIO_41: track 122.1 -> 0.00 mm, vias 4 -> 0
- net /GPIO_39: track 120.0 -> 0.00 mm, vias 2 -> 0
- net /GPIO_17: track 113.4 -> 0.00 mm, vias 5 -> 0
- net GND: track 0.00 -> 62.6 mm, vias 0 -> 6
- net /GPIO_15: track 102.1 -> 153.2 mm
- net /GPIO_16: track 89.7 -> 138.6 mm
- net /GPIO_TX: track 136.0 -> 90.7 mm, vias 2 -> 0
- net /GPIO_5: track 54.0 -> 93.4 mm
- net /GPIO_6: track 51.7 -> 89.2 mm
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- added copper zone on B.Cu, net GND
Other:
- board size 90 x 90 mm -> 95 x 95 mm

Commit message: chore: pcb rework
Parts:
- removed C6: 100nF, Capacitor_SMD:C_0805_2012Metric_Pad1.18x1.45mm_HandSolder
- added MH1: MountingHole_M2, MountingHole:MountingHole_2.2mm_M2_DIN965_Pad, F.Cu at (135.8, 91.3)
- added MH2: MountingHole_M2, MountingHole:MountingHole_2.2mm_M2_DIN965_Pad, F.Cu at (111.6, 91.3)
- added MH3: MountingHole_M2, MountingHole:MountingHole_2.2mm_M2_DIN965_Pad, F.Cu at (123.7, 112.3)
- added R3: 10k, Resistor_SMD:R_0603_1608Metric, F.Cu at (163.8, 124.0)
- added R9: 10k, Resistor_SMD:R_0603_1608Metric, F.Cu at (163.8, 133.3)
- added REF**: MountingHole_2.7mm_M2.5_DIN965_Pad, MountingHole:MountingHole_2.7mm_M2.5_DIN965_Pad, F.Cu at (168.0, 54.0)
- added REF**: MountingHole_2.7mm_M2.5_DIN965_Pad, MountingHole:MountingHole_2.7mm_M2.5_DIN965_Pad, F.Cu at (168.0, 142.6)
- added REF**: MountingHole_2.7mm_M2.5_DIN965_Pad, MountingHole:MountingHole_2.7mm_M2.5_DIN965_Pad, F.Cu at (79.4, 54.0)
- added REF**: MountingHole_2.7mm_M2.5_DIN965_Pad, MountingHole:MountingHole_2.7mm_M2.5_DIN965_Pad, F.Cu at (79.4, 142.6)
- added TP1: GND Testpoint, TestPoint:TestPoint_Pad_D1.5mm, F.Cu at (145.0, 129.8)
- added TP2: VCC Testpoint, TestPoint:TestPoint_Pad_D1.5mm, F.Cu at (140.5, 129.8)
- added TP3: 3.3V Testpoint, TestPoint:TestPoint_Pad_D1.5mm, F.Cu at (142.7, 144.5)
- added TP4: LEDO Testpoint, TestPoint:TestPoint_Pad_D1.5mm, F.Cu at (117.3, 108.7)
- C5: value 100nF -> 1uF
- JP1: footprint Jumper:SolderJumper-2_P1.3mm_Bridged_RoundedPad1.0x1.5mm -> Jumper:SolderJumper-2_P1.3mm_Open_RoundedPad1.0x1.5mm
- R1, R2, R4, R5, R6, R7, R8: footprint Resistor_SMD:R_0805_2012Metric_Pad1.20x1.40mm_HandSolder -> Resistor_SMD:R_0603_1608Metric
- SW1, SW2: footprint Button_Switch_SMD:SW_SPST_FSMSM -> SW_TL3330AF130QG_EWI:SW_TL3330AF130QG_EWI
- moved C10 116.9 mm to (140.0, 98.4), turned to 90 degrees
- moved C9 116.4 mm to (137.8, 106.6), turned to 60 degrees
- moved C11 115.5 mm to (138.4, 89.2), turned to 120 degrees
- moved D2 115.3 mm to (121.9, 117.4), turned to 0 degrees
- moved D13 115.0 mm to (112.6, 114.0), turned to -30 degrees
- moved C8 114.8 mm to (131.8, 112.6), turned to 30 degrees
- moved D3 114.7 mm to (131.6, 115.7), turned to 30 degrees
- moved C12 114.0 mm to (131.8, 84.2), turned to 150 degrees
- moved D12 113.8 mm to (106.3, 106.4), turned to -60 degrees
- moved D4 113.3 mm to (139.2, 109.4), turned to 60 degrees
- moved D11 112.1 mm to (104.7, 96.6), turned to -90 degrees
- moved C7 111.6 mm to (124.2, 115.8), turned to 0 degrees
- moved D5 111.5 mm to (142.6, 100.2), turned to 90 degrees
- moved C13 111.4 mm to (123.7, 82.0), turned to 180 degrees
- moved D10 110.3 mm to (108.1, 87.4), turned to -120 degrees
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Connections:
- C5 pad 1: /RST -> GND
- C5 pad 2: GND -> /RST
- D13 pad 3: unconnected-(D13-DOUT-Pad3) -> Net-(D13-DOUT)
Routing:
- net VCC: track 52.0 -> 224.8 mm
- net GND: track 62.6 -> 179.1 mm, vias 6 -> 299
- net /GPIO_5: track 93.4 -> 46.7 mm
- net /GPIO_6: track 89.2 -> 45.4 mm
- net /GPIO_2: track 97.9 -> 139.3 mm, vias 2 -> 6
- net /GPIO_7: track 84.3 -> 44.6 mm
- net /GPIO_8: track 75.1 -> 41.5 mm
- net /GPIO_16: track 138.6 -> 170.8 mm
- net +3.3V: track 312.7 -> 340.4 mm, vias 6 -> 2
- net Net-(D2-DIN): track 6.16 -> 32.0 mm, vias 1 -> 2
- net /GPIO_14: track 52.6 -> 69.7 mm
- net /GPIO_47: track 67.7 -> 51.1 mm, vias 6 -> 2
- net /GPIO_9: track 85.1 -> 69.2 mm, vias 4 -> 2
- net /RST: track 145.0 -> 130.5 mm
- net /GPIO_TX: track 90.7 -> 104.8 mm, vias 0 -> 2
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Other:
- outline, holes or cut-outs redrawn
- board text added: "3.3V"
- board text added: "BOOT"
- board text added: "GND"
- board text added: "LED OUT"
- board text added: "RESET"
- board text added: "VCC"

Commit message: chore: pcb updates
Parts:
- removed MH1, MH2, MH3: MountingHole_M2, MountingHole:MountingHole_2.2mm_M2_DIN965_Pad
- added 1: , , F.Cu at (116.7, 110.4)
- added 2: , , F.Cu at (130.7, 110.4)
- added 3: , , F.Cu at (137.7, 98.3)
- added 4: , , F.Cu at (130.7, 86.1)
- added 5: , , F.Cu at (116.7, 86.1)
- added ?: , , F.Cu at (109.7, 98.3)
- added REF**: OSHW-Logo_5.7x6mm_Copper, Symbol:OSHW-Logo_5.7x6mm_Copper, F.Cu at (154.9, 55.4)
- added TP10: TestPoint, TestPoint:TestPoint_Pad_D1.5mm, F.Cu at (86.4, 83.3)
- added TP11: TestPoint, TestPoint:TestPoint_Pad_D1.5mm, F.Cu at (86.4, 85.9)
- added TP12: TestPoint, TestPoint:TestPoint_Pad_D1.5mm, F.Cu at (86.4, 88.4)
- added TP5: TestPoint, TestPoint:TestPoint_Pad_D1.5mm, F.Cu at (86.4, 70.6)
- added TP6: TestPoint, TestPoint:TestPoint_Pad_D1.5mm, F.Cu at (86.4, 73.2)
- added TP7: TestPoint, TestPoint:TestPoint_Pad_D1.5mm, F.Cu at (86.4, 75.7)
- added TP8: TestPoint, TestPoint:TestPoint_Pad_D1.5mm, F.Cu at (86.4, 78.2)
- added TP9: TestPoint, TestPoint:TestPoint_Pad_D1.5mm, F.Cu at (86.4, 80.8)
- J4: value Conn_01x07 -> Conn_01x08
- SW3: footprint Button_Switch_THT:SW_PUSH-12mm -> Button_Switch_THT:SW_PUSH_6mm_H4.3mm
- moved TP4 25.6 mm to (91.9, 111.5)
- moved SW3 3.00 mm to (120.4, 96.0)
- moved U3 2.54 mm to (124.0, 131.8)
- moved R4 1.60 mm to (150.9, 137.7)
- moved R1 1.27 mm to (122.4, 135.4)
- moved R2 1.27 mm to (125.7, 135.4)
- moved JP1 1.20 mm to (155.2, 137.7)
- moved TP3 1.02 mm to (142.7, 143.5)
- moved C15 0.91 mm to (109.0, 89.8)
- moved C12 0.78 mm to (132.2, 83.6)
- moved C13 0.76 mm to (123.7, 81.3)
- moved C7 0.74 mm to (123.7, 115.3)
- moved C10 0.72 mm to (140.7, 98.3)
- moved C14 0.71 mm to (115.2, 83.6)
- moved C9 0.65 mm to (138.4, 106.8)
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Connections:
- net /GPIO_15 renamed /HALL_SENSOR_1
- net /GPIO_16 renamed /HALL_SENSOR_2
- net /GPIO_18 renamed /LIGHT_SENSOR
- net /GPIO_2 renamed /TEMP_SENSOR
- net /GPIO_47 renamed /CLICK_BTN
- net /GPIO_48 renamed /LED_DATA
- J4 pad 3: /GPIO_4 -> /RST
- J4 pad 4: /GPIO_5 -> /LCD_SCK
- J4 pad 5: /GPIO_6 -> /LCD_SDA
- J4 pad 6: /GPIO_7 -> /LCD_BACKLIGHT
- J4 pad 7: /GPIO_8 -> /LCD_CS
- J4 pad 8: /RST -> /LCD_DC
- U1 pad 12: /GPIO_8 -> /LCD_BACKLIGHT
- U1 pad 4: /GPIO_4 -> /LCD_SCK
- U1 pad 5: /GPIO_5 -> /LCD_SDA
- U1 pad 6: /GPIO_6 -> /LCD_DC
- U1 pad 7: /GPIO_7 -> /LCD_CS
Routing:
- net GND: track 179.1 -> 301.2 mm, vias 299 -> 292
- net /LCD_SCK: track 0.00 -> 71.1 mm, vias 0 -> 2
- net /LCD_SDA: track 0.00 -> 66.3 mm, vias 0 -> 2
- net /LCD_BACKLIGHT: track 0.00 -> 60.3 mm, vias 0 -> 4
- net /LCD_CS: track 0.00 -> 57.4 mm, vias 0 -> 2
- net /LCD_DC: track 0.00 -> 55.7 mm, vias 0 -> 2
- net /GPIO_4: track 47.9 -> 0.00 mm, vias 2 -> 0
- net /GPIO_5: track 46.7 -> 0.00 mm, vias 2 -> 0
- net /GPIO_6: track 45.4 -> 0.00 mm, vias 2 -> 0
- net /GPIO_7: track 44.6 -> 0.00 mm, vias 2 -> 0
- net /GPIO_8: track 41.5 -> 0.00 mm, vias 2 -> 0
- net /RST: track 130.5 -> 154.8 mm
- net /HALL_SENSOR_2: track 170.8 -> 193.4 mm
- net /HALL_SENSOR_1: track 164.1 -> 185.9 mm
- net Net-(D13-DOUT): track 8.40 -> 24.7 mm, vias 2 -> 0
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Other:
- board text added: "BL"
- board text added: "CS"
- board text added: "DC"
- board text added: "HS1"
- board text added: "HS2"
- board text added: "IO09"
- board text added: "IO10"
- board text added: "IO11"
- board text added: "IO12"
- board text added: "IO13"
- board text added: "IO14"
- board text added: "RST"
- board text added: "RX"
- board text added: "SCK"
- board text added: "SDA"
- board text added: "TX"

Commit message: chore: pcb updates
Parts:
- added ?: , , F.Cu at (110.7, 103.6)
- moved U5 10.5 mm to (153.9, 130.3)
- moved ? 5.41 mm to (110.7, 93.0)
Routing:
- net /LED_DATA: track 75.3 -> 86.0 mm, vias 2 -> 4
- net +3.3V: track 353.8 -> 345.4 mm, vias 2 -> 4
- net Net-(D2-DIN): track 34.4 -> 42.4 mm
- net VCC: track 236.9 -> 241.6 mm
- net GND: track 301.2 -> 302.8 mm, vias 292 -> 289
Other:
- outline, holes or cut-outs redrawn
- board text added: "SUPPORT MOUNT"

Commit message: pcb updates
Parts:
- added REF**: OSHW-Logo_5.7x6mm_Copper, Symbol:OSHW-Logo_5.7x6mm_Copper, F.Cu at (166.8, 70.2)
- added SW4: BOOT, SMD_SIDED_TACT_SWITCH:SMD_TACT_SWITCH, F.Cu at (163.1, 124.2)
- added SW5: RESET, SMD_SIDED_TACT_SWITCH:SMD_TACT_SWITCH, F.Cu at (163.1, 133.6)
- SW1, SW2: footprint SW_TL3330AF130QG_EWI:SW_TL3330AF130QG_EWI -> SMD_SIDED_TACT_SWITCH:SMD_SIDED_TACT_SWITCH
- moved REF** 19.0 mm to (166.8, 70.2)
- moved R3 5.68 mm to (158.2, 125.0)
- moved R9 5.59 mm to (158.2, 133.3)
- moved C5 4.33 mm to (159.5, 129.5)
- moved J4 2.63 mm to (83.3, 98.3)
- moved R1 0.51 mm to (122.4, 135.9)
- moved R2 0.51 mm to (125.7, 135.9)
- moved SW1 0.20 mm to (168.9, 133.3), turned to -90 degrees
- moved SW2 0.20 mm to (168.9, 124.0), turned to -90 degrees
- moved U3 0.12 mm to (124.0, 131.7), turned to 90 degrees
Connections:
- R9 pad 1: /RST -> +3.3V
- R9 pad 2: +3.3V -> /RST
- U3 pad 1: /ESP_USB_D- -> Net-(J1-D--PadA7)
- U3 pad 3: Net-(J1-D--PadA7) -> Net-(J1-D+-PadA6)
- U3 pad 4: Net-(J1-D+-PadA6) -> /ESP_USB_D+
- U3 pad 6: /ESP_USB_D+ -> /ESP_USB_D-
Routing:
- net +3.3V: track 345.4 -> 333.2 mm
- net GND: track 302.8 -> 311.4 mm, vias 289 -> 285
- net /RST: track 154.8 -> 159.8 mm
- net Net-(U1-IO0): track 110.1 -> 113.4 mm
- net Net-(D2-DIN): track 42.4 -> 39.2 mm
- net /LED_DATA: track 86.0 -> 83.9 mm
- net /LCD_DC: track 55.7 -> 57.7 mm
- net /ESP_USB_D-: track 27.9 -> 26.4 mm
- net /LCD_CS: track 57.4 -> 58.7 mm
- net /ESP_USB_D+: track 29.5 -> 28.2 mm
- net /LCD_BACKLIGHT: track 60.3 -> 61.2 mm
- net VCC: track 241.6 -> 242.5 mm
- net /LCD_SDA: track 66.3 -> 67.2 mm
- net /HALL_SENSOR_1: track 185.9 -> 186.7 mm
- net /HALL_SENSOR_2: track 193.4 -> 194.2 mm
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Other:
- outline, holes or cut-outs redrawn
- board text added: "1.0 r1"
- board text added: "3.3v"
- board text added: "Base PCB"
- board text added: "JLCJLCJLCJLC"
