File: hardware/espac-screen/espac-screen - Copia.kicad_pcb (KiCad board)
At the start: 2 copper layers, 35 x 33.3 mm, 20 parts, among them J1 Conn_01x07, J2 GC9A01, Q1 2N7002

Commit message: pcb updates
Routing:
- net GND: track 103.7 -> 92.3 mm, vias 25 -> 29
- net /RST: track 45.6 -> 45.0 mm
- net /SCK: track 51.4 -> 50.9 mm
Other:
- board text removed: "JLCJLCJLCJLC"
